File: AnalogBuck.kicad_sch (KiCad schematic)
At the start: 61 parts, among them U1 TL594, U2 IR2104, U3 ICL7660, U4 OP177

Commit message: sch update
Parts:
- added CD3, CD4: 100nF, Capacitor_THT:C_Disc_D5.0mm_W2.5mm_P2.50mm, symbol Device:C_US
- R109: renamed from R6; value 6.8K -> 10K
- renumbered C10 to C101, C8 to C102, C11 to C103, C7 to C104, C5 to C105, D204 to DQL3, QL2 to QL1, QL1 to QL2, R9 to R101, R8 to R102, R11 to R103, R10 to R104, R13 to R105, R17 to R106, R18 to R107, R7 to R108, R14 to R110, R12 to R111, R1 to R112, RV1 to RV101, RV2 to RV102
Connections:
- net +5V: now also CD4.1
- net -5V: now also CD4.2
- net GND: now also CD3.2
- net VCC: now also CD3.1
Other:
- title: (none) -> ANALOG SYNCHRONUS BUCK
- moved on the sheet: C101, C102, C103, C104, C105, C201, C301, C302, C303, C304, C6, CB1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
